Commit message: new urdf

File: models/bipedal_plateform_no_arms/urdf/robot.urdf (robot description, URDF)
Before this commit: robot urdf, 17 links, 16 joints
Links:
- removed link torso_mesh
- link ankle_subassembly: mass 0.0168168 -> 0.032674; geometry visual mesh filename=package://assets/07534_05x40_catpart.stl; visual mesh filename=package://assets/bearing_15_21_4.stl
- link ankle_subassembly_2: mass 0.0168168 -> 0.032674; geometry visual mesh filename=package://assets/07534_05x40_catpart.stl; visual mesh filename=package://assets/bearing_15_21_4.stl
- link foot_subassembly: geometry collision mesh filename=package://assets/foot.stl; visual mesh filename=package://assets/07534_05x20_catpart.stl
- link foot_subassembly_2: geometry collision mesh filename=package://assets/foot.stl; visual mesh filename=package://assets/07534_05x20_catpart.stl
- link hipx_subassembly: mass 0.794013 -> 1.05831; geometry visual mesh filename=package://assets/bearing_35_72_17.stl; visual mesh filename=package://assets/hipz12.stl
- link hipx_subassemby_sym: mass 0.794016 -> 1.05831; geometry visual mesh filename=package://assets/bearing_35_72_17.stl; visual mesh filename=package://assets/hipz12_sym.stl
- link hipy_subassembly: mass 0.241618 -> 0.451845; geometry visual mesh filename=package://assets/hipxy.stl
- link hipy_subassembly_sym: mass 0.241619 -> 0.451847; geometry visual mesh filename=package://assets/hipxy_sym.stl
- link shin_subassembly: mass 0.593267 -> 0.637285; geometry visual mesh filename=package://assets/0001755650_00mini_000_asm_1_asm_1_asm_00mi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; visual mesh filename=package://assets/0001755650_00mini_000_asm_1_asm_1_asm_00mi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
- link shin_subassembly_sym: mass 0.593266 -> 0.637284; geometry visual mesh filename=package://assets/0001755650_00mini_000_asm_1_asm_1_asm_00mi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; visual mesh filename=package://assets/0001755650_00mini_000_asm_1_asm_1_asm_00mi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
- link tigh_subassembly: mass 2.5804 -> 2.60644; geometry collision mesh filename=package://assets/femur_12.stl; visual mesh filename=package://assets/1_1_02_eb901_558_1.stl
- link tigh_subassembly_sym: mass 2.5804 -> 2.60644; geometry collision mesh filename=package://assets/femur_12_sym.stl; visual mesh filename=package://assets/1_1_02_eb901_558_1.stl
- link torso_subassembly: mass 1.68455 -> 2.90375; geometry visual mesh filename=package://assets/bearing_35_72_17.stl; visual mesh filename=package://assets/bearing_35_72_17.stl
Joints:
- removed joint mesh
- joint anklex_left: limit lower=-3.141592653589793 upper=3.141592653589793 effort=10 velocity=10 -> lower=-0.174533 upper=0.174533 effort=10 velocity=10; origin xyz=8.54872e-15 -0.01594 0.02 rpy=1.5708 -1.56386 -1.68144e-13 -> xyz=0 -0.01594 0.02 rpy=-1.5708 -1.5644 -3.14159
- joint anklex_right: limit lower=-3.141592653589793 upper=3.141592653589793 effort=10 velocity=10 -> lower=-0.174533 upper=0.174533 effort=10 velocity=10; origin xyz=-5.55112e-15 -0.01594 0.02 rpy=1.5708 1.5708 0 -> xyz=-0 -0.01594 0.02 rpy=1.5708 1.5708 0
- joint ankley_left: limit lower=-3.141592653589793 upper=3.141592653589793 effort=10 velocity=10 -> lower=-0.349066 upper=0.174533 effort=10 velocity=10; origin xyz=-4.996e-16 -0.26 -0.02 rpy=-1.8516e-15 -1.64424e-15 -0.955182 -> xyz=-0 -0.26 -0.02 rpy=-0 -0 -0.955185
- joint ankley_right: limit lower=-3.141592653589793 upper=3.141592653589793 effort=10 velocity=10 -> lower=-0.174533 upper=0.349066 effort=10 velocity=10; origin xyz=-0.221803 -0.135659 0.02 rpy=-3.14159 -6.73194e-15 1.16452 -> xyz=-0.221803 -0.135659 0.02 rpy=3.14159 -0 1.16452
- joint foot_left_frame: origin xyz=-6.35351e-08 -0.035 -0.0480606 rpy=-1.5708 1.5708 0 -> xyz=-6.3535e-08 -0.035 -0.0480606 rpy=-1.5708 1.5708 0
- joint foot_right_frame: origin xyz=-6.35351e-08 -0.035 -0.0480606 rpy=-1.5708 1.5708 0 -> xyz=-6.3535e-08 -0.035 -0.0480606 rpy=-1.5708 1.5708 0
- joint hipx_left: limit lower=-3.141592653589793 upper=3.141592653589793 effort=10 velocity=10 -> lower=-0.349066 upper=0.349066 effort=10 velocity=10; origin xyz=-0.01897 0.0289 -0.09689 rpy=0.0666787 0.313077 2.365 -> xyz=-0.01897 0.0289 -0.09689 rpy=0.0525593 0.315669 2.31935
- joint hipx_right: limit lower=-3.141592653589793 upper=3.141592653589793 effort=10 velocity=10 -> lower=-0.349066 upper=0.349066 effort=10 velocity=10
- joint hipy_left: limit lower=-3.141592653589793 upper=3.141592653589793 effort=10 velocity=10 -> lower=-1.0472 upper=1.0472 effort=10 velocity=10; origin xyz=0.012638 0.0276823 -0.112055 rpy=1.65228 -0.597222 2.66793 -> xyz=0.012638 0.0276823 -0.112055 rpy=1.65237 -0.598815 2.66778
- joint hipy_right: limit lower=-3.141592653589793 upper=3.141592653589793 effort=10 velocity=10 -> lower=-1.0472 upper=1.0472 effort=10 velocity=10
- joint hipz_left: limit lower=-3.141592653589793 upper=3.141592653589793 effort=10 velocity=10 -> lower=-0.349066 upper=0.349066 effort=10 velocity=10; origin xyz=-0.000819037 0.13316 0.04164 rpy=-0.0497558 0.132222 1.18484 -> xyz=-0.000819037 0.13316 0.04164 rpy=-0.0454494 0.133755 1.21732
- joint hipz_right: limit lower=-3.141592653589793 upper=3.141592653589793 effort=10 velocity=10 -> lower=-0.349066 upper=0.349066 effort=10 velocity=10
- joint knee_left: limit lower=-3.141592653589793 upper=3.141592653589793 effort=10 velocity=10 -> lower=-0.523599 upper=0.523599 effort=10 velocity=10; origin xyz=-0.17 -0.294449 -0.0305 rpy=2.37199e-15 -8.32366e-17 -1.52464 -> xyz=-0.17 -0.294449 -0.0305 rpy=0 0 -1.52464
- joint knee_right: limit lower=-3.141592653589793 upper=3.141592653589793 effort=10 velocity=10 -> lower=-0.523599 upper=0.523599 effort=10 velocity=10; origin xyz=0.17 0.294449 -0.0305 rpy=3.14159 -1.53593e-13 -0.544439 -> xyz=0.17 0.294449 -0.0305 rpy=3.14159 -0 -0.544439
- joint torso_frame: origin xyz=1.28979e-17 1.37152e-17 -3.20924e-17 rpy=4.10208e-29 5.06304e-15 -3.16699e-29 -> xyz=-0.000116211 -0.000137208 0.11678 rpy=0 0.00352574 -0
